File: Hardware/PSDPDU/PSU.brd (EAGLE design)
At the start: 50 x 50 mm, 12 parts, among them IC2 REG1117, IC4 MC33269D-5.0, IC7 MC33269D-3.3

Commit message: Added Firmware
Parts:
- added U$6, U$7, U$8, U$9: 5V, SparkFun:STAND-OFF
Connections:
- net N$12 renamed VIN
Routing:
- net GND: track 6.61 -> 23.9 mm, vias 83 -> 68
- net 5V: track 52.0 -> 51.4 mm
- net 3.3V: track 46.6 -> 46.1 mm
- net 1.8V: track 32.1 -> 31.6 mm
- net VIN: vias 0 -> 22
- added copper zone on layer 1, net VIN
- added copper zone on layer 16, net VIN
Other:
- board size 50 x 50 mm -> 50.8 x 50.8 mm
Changed lines of the file:
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@@
 <setting verticaltext="up"/>
 </settings>
-<grid distance="0.05" unitdist="inch" unit="mil" style="lines" multiple="1" display="no" altdistance="0.025" altunitdist="inch" altunit="inch"/>
+<grid distance="8" unitdist="mil" unit="mil" style="lines" multiple="1" display="no" altdistance="0.025" altunitdist="inch" altunit="inch"/>
 <layers>
 <layer number="1" name="Top" color="4" fill="1" visible="yes" active="yes"/>
@@
 <layer number="144" name="Drill_legend" color="7" fill="1" visible="yes" active="yes"/>
 <layer number="151" name="HeatSink" color="7" fill="1" visible="yes" active="yes"/>
+<layer number="199" name="Contour" color="7" fill="1" visible="yes" active="yes"/>
 <layer number="200" name="200bmp" color="1" fill="10" visible="yes" active="yes"/>
 <layer number="201" name="201bmp" color="2" fill="10" visible="yes" active="yes"/>
@@
 <plain>
 <text x="38.1508" y="6.1468" size="1.016" layer="21">+ GND</text>
+<wire x1="2.54" y1="0" x2="0" y2="2.54" width="0.254" layer="20" curve="-90"/>
+<wire x1="0" y1="2.54" x2="0" y2="48.26" width="0.254" layer="20"/>
+<wire x1="0" y1="48.26" x2="2.54" y2="50.8" width="0.254" layer="20" curve="-90"/>
+<wire x1="2.54" y1="50.8" x2="48.26" y2="50.8" width="0.254" layer="20"/>
+<wire x1="48.26" y1="50.8" x2="50.8" y2="48.26" width="0.254" layer="20" curve="-90"/>
+<wire x1="50.8" y1="48.26" x2="50.8" y2="2.54" width="0.254" layer="20"/>
+<wire x1="50.8" y1="2.54" x2="48.26" y2="0" width="0.254" layer="20" curve="-90"/>
+<wire x1="48.26" y1="0" x2="2.54" y2="0" width="0.254" layer="20"/>
 </plain>
 <attributes>
@@
 <element name="U$5" library="terrys" package="ESCPOWER" value="ESC_POWER" x="45.72" y="21.59" rot="R180"/>
 <element name="JP1" library="SparkFun" package="1X02_XTRA_BIG" value="" x="40.64" y="3.81" rot="R180"/>
+<element name="U$6" library="SparkFun" package="STAND-OFF" value="5V" x="2.7178" y="47.9298"/>
+<element name="U$7" library="SparkFun" package="STAND-OFF" value="5V" x="48.0314" y="48.133"/>
+<element name="U$8" library="SparkFun" package="STAND-OFF" value="5V" x="2.7178" y="2.8194"/>
+<element name="U$9" library="SparkFun" package="STAND-OFF" value="5V" x="48.0314" y="2.8194"/>
 </elements>
 <signals>
@@
 <wire x1="18.04" y1="15.5" x2="19.16" y2="15.5" width="0.254" layer="1"/>
 <wire x1="19.16" y1="15.5" x2="19.42" y2="15.24" width="0.254" layer="1"/>
-<polygon width="1.016" layer="16">
+<polygon width="0.254" layer="16" rank="6">
 <vertex x="0" y="50.8"/>
 <vertex x="50.8" y="50.8"/>
@@
 <vertex x="0" y="0"/>
 </polygon>
-<polygon width="1.016" layer="1">
+<polygon width="0.254" layer="1" rank="6">
 <vertex x="0" y="50.8"/>
 <vertex x="50.8" y="50.8"/>
@@
 <via x="10.16" y="15.24" extent="1-16" drill="1.1" shape="square"/>
 <via x="10.16" y="17.78" extent="1-16" drill="1.1" shape="square"/>
-<via x="15.24" y="7.62" extent="1-16" drill="1.1" shape="square"/>
-<via x="15.24" y="10.16" extent="1-16" drill="1.1" shape="square"/>
-<via x="15.24" y="12.7" extent="1-16" drill="1.1" shape="square"/>
 <via x="15.24" y="15.24" extent="1-16" drill="1.1" shape="square"/>
 <via x="15.24" y="17.78" extent="1-16" drill="1.1" shape="square"/>
@@
 <via x="15.24" y="35.56" extent="1-16" drill="1.1" shape="square"/>
 <via x="15.24" y="38.1" extent="1-16" drill="1.1" shape="square"/>
-<via x="17.78" y="7.62" extent="1-16" drill="1.1" shape="square"/>
-<via x="17.78" y="10.16" extent="1-16" drill="1.1" shape="square"/>
-<via x="17.78" y="12.7" extent="1-16" drill="1.1" shape="square"/>
-<via x="20.32" y="12.7" extent="1-16" drill="1.1" shape="square"/>
-<via x="20.32" y="10.16" extent="1-16" drill="1.1" shape="square"/>
-<via x="22.86" y="12.7" extent="1-16" drill="1.1" shape="square"/>
-<via x="34.29" y="12.7" extent="1-16" drill="1.1" shape="square"/>
 <via x="41.91" y="12.7" extent="1-16" drill="1.1" shape="square"/>
 <via x="44.45" y="12.7" extent="1-16" drill="1.1" shape="square"/>
 <via x="46.99" y="12.7" extent="1-16" drill="1.1" shape="square"/>
-<via x="34.29" y="10.16" extent="1-16" drill="1.1" shape="square"/>
-<via x="34.29" y="7.62" extent="1-16" drill="1.1" shape="square"/>
 <via x="34.29" y="5.08" extent="1-16" drill="1.1" shape="square"/>
 <via x="34.29" y="2.54" extent="1-16" drill="1.1" shape="square"/>
@@
 <via x="44.45" y="35.56" extent="1-16" drill="1.1" shape="square"/>
 <via x="22.86" y="48.26" extent="1-16" drill="1.1" shape="square"/>
-<via x="25.4" y="48.26" extent="1-16" drill="1.1" shape="square"/>
 <via x="27.94" y="48.26" extent="1-16" drill="1.1" shape="square"/>
-<via x="27.94" y="45.72" extent="1-16" drill="1.1" shape="square"/>
-<via x="25.4" y="45.72" extent="1-16" drill="1.1" shape="square"/>
 <via x="27.94" y="43.18" extent="1-16" drill="1.1" shape="square"/>
 <via x="2.54" y="16.51" extent="1-16" drill="1.1" shape="square"/>
@@
 <via x="46.99" y="7.62" extent="1-16" drill="1.1" shape="square"/>
 <via x="44.45" y="7.62" extent="1-16" drill="1.1" shape="square"/>
+<wire x1="26.93" y1="15.52" x2="26.93" y2="12.96" width="0.4064" layer="1"/>
+<wire x1="26.93" y1="12.96" x2="26.67" y2="12.7" width="0.4064" layer="1"/>
+<wire x1="26.67" y1="12.7" x2="19.05" y2="12.7" width="0.4064" layer="1"/>
+<wire x1="19.05" y1="12.7" x2="19.05" y2="15.24" width="0.4064" layer="1"/>
+<wire x1="19.05" y1="15.24" x2="17.78" y2="15.24" width="0.4064" layer="1"/>
+<wire x1="15.24" y1="15.24" x2="17.76" y2="15.24" width="0.4064" layer="1"/>
+<wire x1="17.76" y1="15.24" x2="18.04" y2="15.52" width="0.4064" layer="1"/>
 </signal>
 <signal name="5V" class="1">
@@
 <via x="29.21" y="29.21" extent="1-16" drill="0.6" shape="square"/>
 <wire x1="29.21" y1="29.21" x2="33.02" y2="29.21" width="1.016" layer="16"/>
-<wire x1="33.02" y1="29.21" x2="44.45" y2="40.64" width="1.016" layer="16"/>
-<wire x1="44.45" y1="40.64" x2="44.45" y2="48.26" width="1.016" layer="16"/>
+<wire x1="33.02" y1="29.21" x2="43.18" y2="39.37" width="1.016" layer="16"/>
+<wire x1="43.18" y1="39.37" x2="43.18" y2="48.26" width="1.016" layer="16"/>
 </signal>
 <signal name="3.3V">
@@
 <via x="27.94" y="33.02" extent="1-16" drill="0.6" shape="square"/>
 <wire x1="27.94" y1="33.02" x2="31.75" y2="33.02" width="1.016" layer="16"/>
-<wire x1="31.75" y1="33.02" x2="41.91" y2="43.18" width="1.016" layer="16"/>
-<wire x1="41.91" y1="43.18" x2="41.91" y2="48.26" width="1.016" layer="16"/>
+<wire x1="31.75" y1="33.02" x2="40.64" y2="41.91" width="1.016" layer="16"/>
+<wire x1="40.64" y1="41.91" x2="40.64" y2="48.26" width="1.016" layer="16"/>
 </signal>
-<signal name="N$12" class="1">
+<signal name="VIN" class="1">
 <contactref element="IC4" pad="3"/>
 <contactref element="U$2" pad="VIN"/>
@@
 <wire x1="39.37" y1="22.86" x2="39.37" y2="24.13" width="2.54" layer="1"/>
 <wire x1="39.37" y1="24.13" x2="41.91" y2="26.67" width="2.54" layer="1"/>
+<polygon width="0.254" layer="16">
+<vertex x="16.51" y="26.67"/>
+<vertex x="39.37" y="26.67"/>
+<vertex x="39.37" y="7.62"/>
+<vertex x="16.51" y="7.62"/>
+</polygon>
+<polygon width="0.254" layer="1">
+<vertex x="16.51" y="26.67"/>
+<vertex x="39.37" y="26.67"/>
+<vertex x="39.37" y="7.62"/>
+<vertex x="16.51" y="7.62"/>
+</polygon>
+<via x="36.83" y="25.4" extent="1-16" drill="1.1" shape="square"/>
+<via x="36.83" y="22.86" extent="1-16" drill="1.1" shape="square"/>
+<via x="36.83" y="20.32" extent="1-16" drill="1.1" shape="square"/>
+<via x="36.83" y="17.78" extent="1-16" drill="1.1" shape="square"/>
+<via x="36.83" y="15.24" extent="1-16" drill="1.1" shape="square"/>
+<via x="36.83" y="12.7" extent="1-16" drill="1.1" shape="square"/>
+<via x="24.765" y="15.24" extent="1-16" drill="1.1" shape="square"/>
+<via x="24.765" y="25.4" extent="1-16" drill="1.1" shape="square"/>
+<via x="18.415" y="10.16" extent="1-16" drill="1.1" shape="square"/>
+<via x="20.955" y="10.16" extent="1-16" drill="1.1" shape="square"/>
+<via x="23.495" y="10.16" extent="1-16" drill="1.1" shape="square"/>
+<via x="26.035" y="10.16" extent="1-16" drill="1.1" shape="square"/>
+<via x="28.575" y="10.16" extent="1-16" drill="1.1" shape="square"/>
+<via x="31.115" y="10.16" extent="1-16" drill="1.1" shape="square"/>
+<via x="33.655" y="10.16" extent="1-16" drill="1.1" shape="square"/>
+<via x="36.195" y="10.16" extent="1-16" drill="1.1" shape="square"/>
+<via x="33.655" y="12.7" extent="1-16" drill="1.1" shape="square"/>
+<via x="33.655" y="15.24" extent="1-16" drill="1.1" shape="square"/>
+<via x="33.655" y="17.78" extent="1-16" drill="1.1" shape="square"/>
+<via x="33.655" y="20.32" extent="1-16" drill="1.1" shape="square"/>
+<via x="33.655" y="22.86" extent="1-16" drill="1.1" shape="square"/>
+<via x="33.655" y="25.4" extent="1-16" drill="1.1" shape="square"/>
 </signal>
 <signal name="1.8V">
@@
 <via x="25.4" y="35.56" extent="1-16" drill="0.6" shape="square"/>
 <wire x1="25.4" y1="35.56" x2="29.21" y2="35.56" width="1.016" layer="16"/>
-<wire x1="29.21" y1="35.56" x2="39.37" y2="45.72" width="1.016" layer="16"/>
-<wire x1="39.37" y1="45.72" x2="39.37" y2="48.26" width="1.016" layer="16"/>
+<wire x1="29.21" y1="35.56" x2="38.1" y2="44.45" width="1.016" layer="16"/>
+<wire x1="38.1" y1="44.45" x2="38.1" y2="48.26" width="1.016" layer="16"/>
 </signal>
 <signal name="RX">
