File: Hardware/PSDPDU/PSU.sch (EAGLE design)
At the start: 12 parts, among them IC2 REG1117, IC4 MC33269D-5.0, IC7 MC33269D-3.3

Commit message: Added Firmware
Connections:
- net N$12 renamed VIN
- net RX: now also QB1.VIN; no longer QB1.RX
- net TX: now also QB1.BATTSENSE; no longer QB1.TX
Changed lines of the file:
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@@
 </segment>
 </net>
-<net name="N$12" class="1">
+<net name="VIN" class="1">
 <segment>
 <pinref part="IC4" gate="G$1" pin="VI"/>
@@
 <wire x1="203.2" y1="96.52" x2="213.36" y2="96.52" width="0.1524" layer="91" style="longdash"/>
 <label x="203.2" y="96.52" size="1.778" layer="95" rot="R180"/>
-<pinref part="QB1" gate="G$1" pin="RX"/>
+<pinref part="QB1" gate="G$1" pin="VIN"/>
 <wire x1="213.36" y1="96.52" x2="215.9" y2="96.52" width="0.1524" layer="91"/>
 </segment>
@@
 <wire x1="203.2" y1="93.98" x2="213.36" y2="93.98" width="0.1524" layer="91" style="longdash"/>
 <label x="203.2" y="93.98" size="1.778" layer="95" rot="R180"/>
-<pinref part="QB1" gate="G$1" pin="TX"/>
+<pinref part="QB1" gate="G$1" pin="BATTSENSE"/>
 <wire x1="213.36" y1="93.98" x2="215.9" y2="93.98" width="0.1524" layer="91"/>
 </segment>
